File: keychain-uv-index.kicad_pcb (KiCad board)
At the start: 2 copper layers, 23.5 x 27.4 mm, 16 parts, among them J1 Conn_01x06_Pin, SW1 SW_Push_Dual, U1 ATtiny85V-10S

Commit message: edited schematics
Parts:
- added C2: 100n, Capacitor_SMD:C_0805_2012Metric, F.Cu at (58.8, 66.4)
- added C3: 100n, Capacitor_SMD:C_0805_2012Metric, F.Cu at (58.8, 69.4)
- added D2: D_Photo, LED_SMD:LED_PLCC-2_3.4x3.0mm_AK, F.Cu at (52.8, 60.5)
- added R1: 3k3, Resistor_SMD:R_0805_2012Metric, F.Cu at (54.3, 66.4)
- added R3: 1M, Resistor_SMD:R_0805_2012Metric, F.Cu at (54.3, 69.3)
- added R4: 1k, Resistor_SMD:R_0805_2012Metric, F.Cu at (54.3, 72.3)
- added U2: LM358, Package_SO:SOIC-8W_5.3x5.3mm_P1.27mm, F.Cu at (54.9, 54.7)
Connections:
- D1 pad 1: Net-(D1-K) -> GND
- U1 pad 2: Temp -> UVsignal

Commit message: finished PCB design
Parts:
- removed the D2 at (70.4, 64.4)
- removed D3, D4, D5, D6: LED, LED_SMD:LED_0805_2012Metric
- removed the R1 at (68.0, 52.8)
- removed the R3 at (81.0, 59.8)
- removed the R4 at (83.7, 59.8)
- removed TH1: 10k, Resistor_SMD:R_0805_2012Metric
- moved R3 19.7 mm to (73.8, 66.0), turned to -90 degrees
- moved U2 18.9 mm to (72.8, 60.8)
- moved C3 17.5 mm to (70.7, 56.6)
- moved D2 16.5 mm to (66.8, 69.3)
- moved R4 14.8 mm to (66.2, 63.3), turned to 90 degrees
- moved D1 11.3 mm to (74.0, 55.5), turned to -90 degrees
- moved R1 11.0 mm to (65.3, 66.2), turned to 180 degrees
- moved C2 10.5 mm to (69.2, 66.2), turned to 180 degrees
- moved C1 9.81 mm to (75.1, 46.2), turned to 180 degrees
- moved U1 5.04 mm to (72.9, 50.2)
- moved R2 4.57 mm to (76.7, 55.5)
- moved J1 3.67 mm to (72.5, 69.8)
Connections:
- D2 pad 2: Net-(D2-A) -> GND
- U2 pad 3: Net-(D2-A) -> GND
Routing:
- net UVsignal: track 0.00 -> 22.2 mm
- net Net-(D1-A): track 23.0 -> 2.63 mm, vias 2 -> 0
- net GND: track 3.74 -> 20.8 mm, vias 3 -> 6
- net Net-(D1-K): track 15.8 -> 0.00 mm
- net Net-(D2-K): track 0.00 -> 14.2 mm
- net Net-(D3-K): track 13.3 -> 0.00 mm
- net Temp: track 13.1 -> 0.00 mm
- net Net-(C2-Pad2): track 0.00 -> 10.8 mm, vias 0 -> 2
- net A: track 14.0 -> 22.0 mm, vias 1 -> 0
- net PB5-reset: track 18.8 -> 25.2 mm
- net C: track 19.4 -> 24.1 mm
- net B: track 18.0 -> 21.8 mm, vias 1 -> 0
- net VCC: track 43.9 -> 45.9 mm
Other:
- outline, holes or cut-outs redrawn
- board text added: "GND"
- board text added: "PB0"
- board text added: "PB1"
- board text added: "PB2"
- board text added: "Reset"
- board text added: "UV index indicator"
- board text added: "Vcc"
- board text removed: "32+16 +8 + 4 + 2 + 1"
- board text removed: "Keychain Thermometer"
